File: ThumbsUp.kicad_pcb (KiCad board)
At the start: 2 copper layers, 211.3 x 232.1 mm, 56 parts, among them J1 52559-1233, J1L1 PJ-3200B, J1R1 PJ-3200B, J2 52559-1233, U1 ProMicro

Commit message: v12: Cleaned up orphaned tracks, prepared for Gerbers generation..
Routing:
- net (no net): track 45.0 -> 0.00 mm
- net GND-P: track 0.00 -> 44.5 mm, vias 0 -> 2
- net GND: track 599.5 -> 602.3 mm
- added copper zone on B.Cu, net GND-P
- added copper zone on F.Cu, net GND-P
